File: VDP.kicad_sch (KiCad schematic)
At the start: 5 parts

Commit message: Migrate to KiCad v8
Parts:
- C1, C2: renamed from C?; value (none) -> 56pF; footprint (none) -> artemisa:Disc_capacitor
- C3: renamed from C?; value (none) -> 100nF; footprint (none) -> artemisa:Disc_capacitor
- U1: renamed from U?; value (none) -> TMS9928; footprint (none) -> artemisa:DIP-40_600
- Y1: renamed from Y?; value (none) -> 10.7386Mhz; footprint (none) -> artemisa:Crystal
