File: VDP.kicad_sch (KiCad schematic)
At the start: 5 parts, among them U1 TMS9928, Y1 10.7386Mhz

Commit message: Update to latest Artemisa kicadlibs
Parts:
- U1: symbol artemisa:TMS9928 -> PCM_artemisa:TMS9928
Connections:
- net RD0 renamed D0
- net RD1 renamed D1
- net RD2 renamed D2
- net RD3 renamed D3
- net RD4 renamed D4
- net RD5 renamed D5
- net RD6 renamed D6
- net RD7 renamed D7
Changed lines of the file:
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@@
 		)
 	)
-	(label "RD5"
+	(label "D5"
 		(at 171.45 104.14 180)
 		(effects
@@
 		)
 	)
-	(label "RD7"
+	(label "D7"
 		(at 171.45 99.06 180)
 		(effects
@@
 		)
 	)
-	(label "RD0"
+	(label "D0"
 		(at 171.45 116.84 180)
 		(effects
@@
 		)
 	)
-	(label "RD4"
+	(label "D4"
 		(at 171.45 106.68 180)
 		(effects
@@
 		)
 	)
-	(label "RD6"
+	(label "D6"
 		(at 171.45 101.6 180)
 		(effects
@@
 		)
 	)
-	(label "RD1"
+	(label "D1"
 		(at 171.45 114.3 180)
 		(effects
@@
 		)
 	)
-	(label "RD3"
+	(label "D3"
 		(at 171.45 109.22 180)
 		(effects
@@
 		)
 	)
-	(label "RD2"
+	(label "D2"
 		(at 171.45 111.76 180)
 		(effects
@@
 		)
 	)
-	(hierarchical_label "RD[0..7]"
+	(hierarchical_label "D[0..7]"
 		(shape input)
 		(at 181.61 97.79 0)
@@
 	)
 	(symbol
-		(lib_id "artemisa:TMS9928")
+		(lib_id "PCM_artemisa:TMS9928")
 		(at 144.78 100.33 0)
 		(unit 1)

Commit message: Use spare MCP6294 as CSYNC buffer
Parts:
- C1, C2, C3: footprint artemisa:Disc_capacitor -> PCM_artemisa:Disc_capacitor
- U1: footprint artemisa:DIP-40_600 -> PCM_artemisa:DIP-40_600
- Y1: footprint artemisa:Crystal -> PCM_artemisa:Crystal
Changed lines of the file:
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@@
 			)
 		)
-		(property "Footprint" "artemisa:Crystal"
+		(property "Footprint" "PCM_artemisa:Crystal"
 			(at 118.11 116.84 0)
 			(hide yes)
@@
 			)
 		)
-		(property "Footprint" "artemisa:Disc_capacitor"
+		(property "Footprint" "PCM_artemisa:Disc_capacitor"
 			(at 107.95 111.76 0)
 			(hide yes)
@@
 			)
 		)
-		(property "Footprint" "artemisa:Disc_capacitor"
+		(property "Footprint" "PCM_artemisa:Disc_capacitor"
 			(at 107.95 121.92 0)
 			(hide yes)
@@
 			)
 		)
-		(property "Footprint" "artemisa:Disc_capacitor"
+		(property "Footprint" "PCM_artemisa:Disc_capacitor"
 			(at 149.86 54.61 0)
 			(hide yes)
@@
 			)
 		)
-		(property "Footprint" "artemisa:DIP-40_600"
+		(property "Footprint" "PCM_artemisa:DIP-40_600"
 			(at 144.78 86.36 0)
 			(hide yes)
