File: gfx-9920.kicad_pcb (KiCad board)
At the start: 2 copper layers, 50 x 150 mm, 28 parts, among them J1 GFX_Connector_Input, J2 RCA_Conn, J3 RCA_Conn, J4 RCA_Conn, U1 TMS9918, U2 74HCT04, U3 74HCT574, U4 74HCT574, U5 74HCT574, U6 62256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

Commit message: Migrate to KiCad v6
Connections:
- net /Input connector & power/~INT renamed /Input connector & power/~{INT}
- net /Input connector & power/~RD renamed /Input connector & power/~{RD}
- net /Input connector & power/~RESET renamed /Input connector & power/~{RESET}
- net /Input connector & power/~VDPIOSL renamed /Input connector & power/~{VDPIOSL}
- net /Input connector & power/~WR renamed /Input connector & power/~{WR}
- net /Interface Decoding Logic/~CSW renamed /Interface Decoding Logic/~{CSW}
- net /VRAM Decoding Logic/~CAS renamed /VRAM Decoding Logic/~{CAS}
- net /VRAM Decoding Logic/~RAS renamed /VRAM Decoding Logic/~{RAS}
- net /VRAM Decoding Logic/~WR renamed /VRAM Decoding Logic/~{WR}
Other:
- net class Default removed
- net class Power removed
