File: video-encoding.kicad_sch (KiCad schematic)
At the start: 48 parts

Commit message: Migrate to KiCad v8
Parts:
- C10, C15: renamed from C?; value (none) -> 100nF; footprint (none) -> artemisa:Disc_capacitor
- C12: renamed from C?; value (none) -> 10nF; footprint (none) -> artemisa:Disc_capacitor
- C13, C14: renamed from C?; value (none) -> 100nF
- J2: value (none) -> DIN8
- Q1: value (none) -> 2N2222
- R1, R2, R3: value (none) -> 470
- R10: renamed from R?; value (none) -> 680K
- R11, R12, R13, R15, R27: renamed from R?; value (none) -> 180
- R14, R16, R7, R8, R9: renamed from R?; value (none) -> 360
- R17, R24, R5: renamed from R?; value (none) -> 1K
- R18, R20, R21, R22, R23, R26: renamed from R?; value (none) -> 200
- R19, R25: renamed from R?; value (none) -> 240
- R28, R29, R30, R31: renamed from R?; value (none) -> 75
- R36: renamed from R?; value (none) -> 680
- R4, R6: value (none) -> 10K
- U10, U11, U12, U14, U15, U16, U9: renamed from U?; value (none) -> LM318
- U13: renamed from U?; value (none) -> LM1881
- U8: value (none) -> 4066
