File: vram-decoding.kicad_sch (KiCad schematic)
At the start: 12 parts

Commit message: Migrate to KiCad v8
Parts:
- C5, C6, C7: renamed from C?; value (none) -> 100nF; footprint (none) -> artemisa:Disc_capacitor
- U2: renamed from U?; value (none) -> 74HCT04; footprint (none) -> artemisa:DIP-14_300
- U3, U4, U5: renamed from U?; value (none) -> 74HCT574; footprint (none) -> artemisa:DIP-20_300
