File: vram.kicad_sch (KiCad schematic)
At the start: 2 parts

Commit message: Migrate to KiCad v8
Parts:
- C4: renamed from C?; value (none) -> 100nF; footprint (none) -> artemisa:Disc_capacitor
- U6: renamed from U?; value (none) -> 62256; footprint (none) -> artemisa:DIP-28_600
